Commit message: 개선 알고리즘 반영

File: my_robot_description/urdf/my_robot.urdf (robot description, URDF)
Before this commit: robot tracking_robot, 5 links, 4 joints
Joints:
- joint left_wheel_joint: origin xyz=0.05 0.105 -0.01 rpy=-1.5708 0 0 -> xyz=0.05 0.092 -0.01 rpy=-1.5708 0 0
- joint right_wheel_joint: origin xyz=0.05 -0.105 -0.01 rpy=-1.5708 0 0 -> xyz=0.05 -0.092 -0.01 rpy=-1.5708 0 0
